File: hardware/woofii/woofii.kicad_pcb (KiCad board)
At the start: 2 copper layers, 20.3 x 50.8 mm, 28 parts, among them J1 Conn_01x10, J2 Conn_01x10, U1 ap6212a, Y1 26M

Commit message: WooFii: Clean up pcb layout.
Routing:
- net /sdio_d1: track 14.7 -> 15.9 mm
- net /sdio_d2: track 22.5 -> 23.6 mm
- net /bt_wake: track 20.7 -> 19.8 mm
- net /sdio_d3: track 24.6 -> 25.3 mm
- net GND: track 53.0 -> 52.5 mm
