File: hardware/woofii/woofii.sch (KiCad schematic (older format))
At the start: 28 parts, among them J1 Conn_01x10, J2 Conn_01x10, U1 ap6212a, Y1 26M

Commit message: Defconfig and env tweaks
Parts:
- C4: value C -> 4.7uf
Changed lines of the file:
@@
 P 5850 1700
 F 0 "C4" H 5965 1746 50  0000 L CNN
-F 1 "C" H 5965 1655 50  0000 L CNN
+F 1 "4.7uf" H 5965 1655 50  0000 L CNN
 F 2 "Capacitor_SMD:C_0603_1608Metric" H 5888 1550 50  0001 C CNN
 F 3 "~" H 5850 1700 50  0001 C CNN
