File: hardware/doge/bucksupply.sch (KiCad schematic (older format))
At the start: 7 parts, among them U3 RT8059GJ5

Commit message: DogeDoge Rev1: switch ldo for xc6204, expose en single on buck supplies, tie enables together
Parts:
- added R?: R, symbol Device:R
Connections:
- net labels added: en
- wire segments 29 -> 32
Changed lines of the file:
@@
 $Descr A4 11693 8268
 encoding utf-8
-Sheet 3 5
+Sheet 2 5
 Title ""
 Date ""
@@
 AR Path="/5B8FA736/5B851B00" Ref="U4"  Part="1"
 AR Path="/5B8FA7CE/5B851B00" Ref="U5"  Part="1"
-F 0 "U4" H 5250 3865 50  0000 C CNN
+F 0 "U3" H 5250 3865 50  0000 C CNN
 F 1 "RT8059GJ5" H 5250 3774 50  0000 C CNN
 F 2 "Package_TO_SOT_SMD:TSOT-23-5" H 5250 3450 50  0001 C CNN
@@
 L Device:C C?
 U 1 1 5B851BD5
-P 4400 3550
+P 4400 3500
 AR Path="/665FBD11/5B851806/5B851BD5" Ref="C?"  Part="1"
 AR Path="/665FBD11/5B972AC4/5B851BD5" Ref="C?"  Part="1"
@@
 AR Path="/5B8FA736/5B851BD5" Ref="C10"  Part="1"
 AR Path="/5B8FA7CE/5B851BD5" Ref="C13"  Part="1"
-F 0 "C10" H 4515 3596 50  0000 L CNN
-F 1 "4.7uF" H 4515 3505 50  0000 L CNN
-F 2 "Capacitor_SMD:C_0603_1608Metric" H 4438 3400 50  0001 C CNN
-F 3 "~" H 4400 3550 50  0001 C CNN
-	1    4400 3550
-	1    0    0    -1
-$EndComp
-Wire Wire Line
-	4750 3300 4650 3300
-Wire Wire Line
-	4400 3300 4400 3400
+F 0 "C7" H 4150 3600 50  0000 L CNN
+F 1 "4.7uF" H 4050 3500 50  0000 L CNN
+F 2 "Capacitor_SMD:C_0603_1608Metric" H 4438 3350 50  0001 C CNN
+F 3 "~" H 4400 3500 50  0001 C CNN
+	1    4400 3500
+	1    0    0    -1
+$EndComp
+Wire Wire Line
+	4400 3300 4400 3350
 Connection ~ 4400 3300
 Wire Wire Line
@@
 	4750 3550 4650 3550
 Wire Wire Line
-	4650 3550 4650 3300
-Connection ~ 4650 3300
-Wire Wire Line
-	4650 3300 4400 3300
-Wire Wire Line
-	4400 3700 4400 4250
-Wire Wire Line
-	4400 4250 5250 4250
+	4400 3650 4400 4250
+Wire Wire Line
+	4400 4250 4650 4250
 Wire Wire Line
 	5250 4250 5250 3950
@@
 AR Path="/5B8FA736/5B851CF1" Ref="L2"  Part="1"
 AR Path="/5B8FA7CE/5B851CF1" Ref="L3"  Part="1"
-F 0 "L2" V 6190 3300 50  0000 C CNN
+F 0 "L1" V 6190 3300 50  0000 C CNN
 F 1 "L" V 6099 3300 50  0000 C CNN
 F 2 "cd32:CD32" H 6000 3300 50  0001 C CNN
@@
 AR Path="/5B8FA736/5B851DC3" Ref="C11"  Part="1"
 AR Path="/5B8FA7CE/5B851DC3" Ref="C14"  Part="1"
-F 0 "C11" H 6365 3546 50  0000 L CNN
+F 0 "C8" H 6365 3546 50  0000 L CNN
 F 1 "C" H 6365 3455 50  0000 L CNN
 F 2 "Capacitor_SMD:C_0603_1608Metric" H 6288 3350 50  0001 C CNN
@@
 AR Path="/5B8FA736/5B851E28" Ref="R6"  Part="1"
 AR Path="/5B8FA7CE/5B851E28" Ref="R8"  Part="1"
-F 0 "R6" H 6620 3546 50  0000 L CNN
+F 0 "R4" H 6620 3546 50  0000 L CNN
 F 1 "R" H 6620 3455 50  0000 L CNN
 F 2 "Resistor_SMD:R_0603_1608Metric" V 6480 3500 50  0001 C CNN
@@
 AR Path="/5B8FA736/5B851E80" Ref="R7"  Part="1"
 AR Path="/5B8FA7CE/5B851E80" Ref="R9"  Part="1"
-F 0 "R7" H 6620 3946 50  0000 L CNN
+F 0 "R5" H 6620 3946 50  0000 L CNN
 F 1 "R" H 6620 3855 50  0000 L CNN
 F 2 "Resistor_SMD:R_0603_1608Metric" V 6480 3900 50  0001 C CNN
@@
 AR Path="/5B8FA736/5B851EE7" Ref="C12"  Part="1"
 AR Path="/5B8FA7CE/5B851EE7" Ref="C15"  Part="1"
-F 0 "C12" H 6915 3746 50  0000 L CNN
+F 0 "C9" H 6915 3746 50  0000 L CNN
 F 1 "10uF" H 6915 3655 50  0000 L CNN
 F 2 "Capacitor_SMD:C_0603_1608Metric" H 6838 3550 50  0001 C CNN
@@
 	6800 3300 7000 3300
 Connection ~ 6800 3300
+$Comp
+L Device:R R?
+U 1 1 5BBF42E7
+P 4650 3900
+AR Path="/5B8FA608/5BBF42E7" Ref="R?"  Part="1"
+AR Path="/5B8FA736/5BBF42E7" Ref="R?"  Part="1"
+AR Path="/5B8FA7CE/5BBF42E7" Ref="R?"  Part="1"
+F 0 "R?" H 4720 3946 50  0000 L CNN
+F 1 "R" H 4720 3855 50  0000 L CNN
+F 2 "" V 4580 3900 50  0001 C CNN
+F 3 "~" H 4650 3900 50  0001 C CNN
+	1    4650 3900
+	1    0    0    -1
+$EndComp
+Wire Wire Line
+	4650 4050 4650 4250
+Connection ~ 4650 4250
+Wire Wire Line
+	4650 4250 5250 4250
+Wire Wire Line
+	4400 3300 4750 3300
+Wire Wire Line
+	4650 3550 4650 3700
+Wire Wire Line
+	4150 3700 4650 3700
+Connection ~ 4650 3700
+Wire Wire Line
+	4650 3700 4650 3750
+Text HLabel 4150 3700 0    50   Input ~ 0
+en
 $EndSCHEMATC
