File: hardware/doge/doge.sch (KiCad schematic (older format))
At the start: 51 parts, among them J1 Conn_01x22, J2 Conn_01x22, J4 Conn_01x05, J5 Conn_01x05, J6 Conn_01x15, U1 vs3, U2 AMS1117-3.3, U6 spinor, Y1 24MHz, Y2 32KHz

Commit message: DogeDoge Rev1: switch ldo for xc6204, expose en single on buck supplies, tie enables together
Parts:
- removed U2: AMS1117-3.3, Package_TO_SOT_SMD:SOT-23, symbol Regulator_Linear:AMS1117-3.3
- added R?: R, symbol Device:R
- added U2: xc6204xxxxMR, symbol xc6204:xc6204xxxxMR
Connections:
- wire segments 438 -> 444
